Commit message: Attempting reinstall of ROSSHARP

File: rover_sim/Assets/dev_arm/urdf/dev_arm.urdf (robot description, URDF)
Before this commit: robot dev_arm, 9 links, 8 joints
Links:
- removed link link_ee
- added link ee_base_link
- added link finger_left, mass 0.115999619262241; collision mesh filename=package://dev_arm/meshes/finger_left.STL; visual mesh filename=package://dev_arm/meshes/finger_left.STL
- added link finger_right, mass 0.115999628451242; collision mesh filename=package://dev_arm/meshes/finger_right.STL; visual mesh filename=package://dev_arm/meshes/finger_right.STL
Joints:
- added joint finger_left_joint: type prismatic, parent ee_base_link, child finger_right, origin xyz=-0.23241 0.37651 0.0074738 rpy=-3.0542 -0.36707 2.5976, axis -0.32112 0.14724 0.93552, limit lower=-0.0325 upper=0.061 effort=1 velocity=1
- added joint finger_right_joint: type prismatic, parent ee_base_link, child finger_left, origin xyz=-0.25101 0.39517 0.094886 rpy=-0.087358 0.36707 -0.54398, axis 0.32112 0.14724 -0.93552, limit lower=-0.061 upper=0.0325 effort=1 velocity=1
- joint joint_ee: child link_ee -> ee_base_link; origin xyz=-0.073337 -0.033291 0.14226 rpy=-3.1416 0 1.6469 -> xyz=0.0 0.0145 0.078 rpy=0 -1.5707963 0
